File: RPiProject.sch (EAGLE design)
At the start: 32 parts

Commit message: version 2
Parts:
- removed C5: 100uF, SparkFun-Retired:100UF6.3V20%(1210)
- removed C6: (no value), rcl:C-US050-030X075
- removed D3: (no value), eagle-ltspice:SCHOTTKY-DIODE
- removed ENCODERL, ENCODERR, LOCALINO: (no value), ee2parts:R
- removed IC1, IC3, IC4, IC5: (no value), LM2576:LM2576-T05A
- removed L3: (no value), resistor:L-US0207/7
- added LM2576-3.3A, LM2576-5.0A, LM2576-5.0B: (no value), LM2576:LM2576-T05A
- added U$2, U$3: ENCODER_A6B2, RaspberryPi:ENCODER_A6B2
- renumbered U$4 to NEATOXV11LIDAR
Connections:
- removed net N$14: C12.1, C8.1, IC5.FB, L5.2, NEATOXV11LIDAR.VDD, NEATOXV11LIDAR.VDDIO, R1.2, R2.2, U$6.PWR
- removed net N$18: ENCODERL.2
- removed net N$19: ENCODERR.2
- removed net N$7: C10.1, IC4.FB, L4.2, U$6.+5V
- new net N$20: D5.A, L5.1, LM2576-3.3A.+V_OUT
- new net N$21: D4.A, L4.1, LM2576-5.0A.+V_OUT
- new net N$4: C10.1, L4.2, LM2576-5.0A.FB, U$2.BROWN_VCC, U$3.BROWN_VCC, U$6.+5V
- net GND: now also LM2576-5.0B.GND, LM2576-5.0B._EN/DIS, U$2.BLUE_0V, U$2.SMELD_GND, U$3.BLUE_0V, U$3.SMELD_GND; no longer ENCODERL.1, ENCODERR.1, IC1.GND, IC1._EN/DIS, LOCALINO.1
- net GND2: now also LM2576-3.3A.GND, LM2576-3.3A._EN/DIS, LM2576-5.0A.GND, LM2576-5.0A._EN/DIS; no longer C5.2, C6.2, D3.C, IC3.GND, IC3._EN/DIS, IC4.GND, IC4._EN/DIS, IC5.GND, IC5._EN/DIS
- net N$2: now also LM2576-5.0B.FB; no longer IC1.FB
- net N$3: now also LM2576-5.0B.+V_OUT; no longer IC1.+V_OUT
- net N$5: now also C12.1, C8.1, L5.2, LM2576-3.3A.FB, NEATOXV11LIDAR.VDD, NEATOXV11LIDAR.VDDIO, R1.2, R2.2, U$6.PWR; no longer C6.1, IC3.FB, L3.2, LOCALINO.2
- net VCC: now also LM2576-3.3A.+V_IN, LM2576-5.0A.+V_IN, LM2576-5.0B.+V_IN; no longer C5.1, IC1.+V_IN, IC3.+V_IN, IC4.+V_IN, IC5.+V_IN
Other:
- note added: "5V @ 2.5A"
- note added: "5V @ 535mA"
- note added: "DC-DC Converters"
- moved on the sheet: C1, C10, C11, C12, C4, C9, D1, D4, D5, L1, L4, L5
